Commit message: 1st_trail-zyx

File: resources/robots/hi/urdf/hi_23dof_250401_rl.urdf (robot description, URDF)
Before this commit: robot hi_23dof_250401, 27 links, 26 joints
Links:
- link l_hip_pitch_link: geometry collision box size=0.06 0.37 0.06; visual mesh filename=../meshes/l_hip_pitch_link.STL
- link l_thigh_link: geometry collision box size=0.01 0.01 0.11; visual mesh filename=../meshes/l_thigh_link.STL
- link r_hip_pitch_link: geometry collision box size=0.06 0.37 0.06; visual mesh filename=../meshes/r_hip_pitch_link.STL
- link r_thigh_link: geometry collision box size=0.01 0.01 0.11; visual mesh filename=../meshes/r_thigh_link.STL
Joints:
- joint l_ankle_pitch_joint: origin xyz=0 0.00475 -0.2 rpy=0 0 0 -> xyz=0 0.00475 -0.3 rpy=0 0 0
- joint l_calf_joint: origin xyz=0 0.00375 -0.069 rpy=0 0 0 -> xyz=0 0.00375 -0.169 rpy=0 0 0
- joint l_hip_roll_joint: origin xyz=0.02725 0.042 0 rpy=0 0 0 -> xyz=0.02725 0.072 0 rpy=0 0 0
- joint r_ankle_pitch_joint: origin xyz=0 -0.00475 -0.2 rpy=0 0 0 -> xyz=0 -0.00475 -0.3 rpy=0 0 0
- joint r_calf_joint: origin xyz=0 -0.00375 -0.069 rpy=0 0 0 -> xyz=0 -0.00375 -0.169 rpy=0 0 0
- joint r_hip_roll_joint: origin xyz=0.02725 -0.042 0 rpy=0 0 0 -> xyz=0.02725 -0.072 0 rpy=0 0 0

Commit message: 1st_trail-zyx

File: resources/robots/hi/urdf/hi_23dof_250401_rl.urdf (robot description, URDF)
Before this commit: robot hi_23dof_250401, 27 links, 26 joints
Links:
- link l_calf_link: geometry collision box size=0.06 0.06 0.19; visual mesh filename=../meshes/l_calf_link.STL
- link l_hip_pitch_link: geometry collision box size=0.06 0.10 0.06; visual mesh filename=../meshes/l_hip_pitch_link.STL
- link l_thigh_link: geometry collision box size=0.05 0.05 0.11; visual mesh filename=../meshes/l_thigh_link.STL
- link r_calf_link: geometry collision box size=0.06 0.06 0.19; visual mesh filename=../meshes/r_calf_link.STL
- link r_hip_pitch_link: geometry collision box size=0.06 0.10 0.06; visual mesh filename=../meshes/r_hip_pitch_link.STL
- link r_thigh_link: geometry collision box size=0.05 0.05 0.11; visual mesh filename=../meshes/r_thigh_link.STL
